Commit message: first commit

File: src/lauv_description/robots/default.xacro (robot description, xacro)
@@ -3,9 +3,12 @@
   <xacro:arg name="debug" default="0"/>
   <xacro:arg name="namespace" default="lauv"/>
+  <xacro:arg name="inertial_reference_frame" default="world"/>
   <!-- Include the ROV macro file -->
   <xacro:include filename="$(find lauv_description)/urdf/base.xacro"/>
   <xacro:include filename="$(find lauv_description)/urdf/gazebo.xacro"/>
   <!-- Create the lauv -->
-  <xacro:lauv_base namespace="$(arg namespace)">
+  <xacro:lauv_base
+    namespace="$(arg namespace)"
+    inertial_reference_frame="$(arg inertial_reference_frame)">
     <!-- The underwater object plugin is given as an input block parameter to
      allow the addition of external models of manipulator units -->

File: src/lauv_description/urdf/actuators.xacro (robot description, xacro)
@@ -9,24 +9,18 @@
     -->
     <xacro:thruster_macro robot_namespace="${namespace}" thruster_id="0">
-        <origin xyz="0 0 0" rpy="0 0 ${pi}" />
-    </xacro:thruster_macro>
-    <xacro:thruster_macro robot_namespace="${namespace}" thruster_id="1">
-        <origin xyz="0 0 0" rpy="0 0 ${pi}" />
-    </xacro:thruster_macro>
-    <xacro:thruster_macro robot_namespace="${namespace}" thruster_id="2">
-    <origin xyz="0 0 0" rpy="0 -${0.5*pi} 0" />
+        <origin xyz="-0.53994 0 0" rpy="0 0 ${pi}" />
     </xacro:thruster_macro>
     <!-- Instantiate fins, if necessary -->
-    <xacro:fin_macro namespace="${namespace}" fin_id="0">
-      <origin xyz="0 0 0" rpy="0 0 0" />
+    <xacro:fin_macro namespace="${namespace}" fin_id="0" mesh_filename="${red_fin_mesh_file}">
+      <origin xyz="-0.4 0 0.04" rpy="0 0 0" />
     </xacro:fin_macro>
-    <xacro:fin_macro namespace="${namespace}" fin_id="1">
-      <origin xyz="0 0 0" rpy="0 0 0" />
+    <xacro:fin_macro namespace="${namespace}" fin_id="1" mesh_filename="${black_fin_mesh_file}">
+      <origin xyz="-0.4 -0.04 0" rpy="${0.5 * pi} 0 0" />
     </xacro:fin_macro>
-    <xacro:fin_macro namespace="${namespace}" fin_id="2">
-      <origin xyz="0 0 0" rpy="0 0 0" />
+    <xacro:fin_macro namespace="${namespace}" fin_id="2" mesh_filename="${black_fin_mesh_file}">
+      <origin xyz="-0.4 0 -0.04" rpy="${pi} 0 0" />
     </xacro:fin_macro>
-    <xacro:fin_macro namespace="${namespace}" fin_id="3">
-      <origin xyz="0 0 0" rpy="0 0 0" />
+    <xacro:fin_macro namespace="${namespace}" fin_id="3" mesh_filename="${black_fin_mesh_file}">
+      <origin xyz="-0.4 0.04 0" rpy="${-0.5 * pi} 0 0" />
     </xacro:fin_macro>
 </robot>

File: src/lauv_description/urdf/base.xacro (robot description, xacro)
@@ -12,5 +12,5 @@
     Vehicle's parameters (remember to enter the model parameters below)
   -->
-  <xacro:property name="mass" value="0"/>
+  <xacro:property name="mass" value="18"/>
   <!-- Center of gravity -->
   <xacro:property name="cog" value="0 0 0"/>
@@ -23,11 +23,11 @@
     Open the meshes for the RexROV vehicle in Blender to see an example on the mesh placement.
   -->
-  <xacro:property name="visual_mesh_file" value="file://$(find lauv_description)/meshes/vehicle.dae"/>
+  <xacro:property name="visual_mesh_file" value="file://$(find lauv_description)/meshes/body.dae"/>
   <!-- Collision geometry mesh, usually in STL format (it is recommended to keep
   this geometry as simple as possible to improve the performance the physics engine
   regarding the computation of collision forces) -->
-  <xacro:property name="collision_mesh_file" value="file://$(find lauv_description)/meshes/vehicle.stl"/>
+  <xacro:property name="collision_mesh_file" value="file://$(find lauv_description)/meshes/body.stl"/>
   <!-- Vehicle macro -->
-  <xacro:macro name="lauv_base" params="namespace *gazebo">
+  <xacro:macro name="lauv_base" params="namespace *gazebo inertial_reference_frame">
       <!-- Rigid body description of the base link -->
       <link name="${namespace}/base_link">
@@ -39,7 +39,7 @@
           <mass value="${mass}" />
           <origin xyz="${cog}" rpy="0 0 0"/>
-          <inertia ixx="0" ixy="0" ixz="0"
-                   iyy="0" iyz="0"
-                   izz="0" />
+          <inertia ixx="${0.5 * mass * lauv_radius * lauv_radius}" ixy="0" ixz="0"
+                   iyy="${0.083333333 * mass * 3 * lauv_radius * lauv_radius + 0.083333333 * mass * lauv_length * lauv_length}" iyz="0"
+                   izz="${0.083333333 * mass * 3 * lauv_radius * lauv_radius + 0.083333333 * mass * lauv_length * lauv_length}" />
         </inertial>
         <visual>
@@ -50,5 +50,5 @@
         </visual>
         <collision>
-          <origin xyz="0 0 0" rpy="0 0 0"/>
+          <origin xyz="0 0 0" rpy="0 0 0"/>s
           <geometry>
             <mesh filename="${collision_mesh_file}" scale="1 1 1" />

File: src/lauv_description/urdf/gazebo.xacro (robot description, xacro)
@@ -2,11 +2,12 @@
 <robot xmlns:xacro="http://www.ros.org/wiki/xacro">
     <!-- Center of buoyancy -->
-    <xacro:property name="lauv_cob" value="0 0 0"/>
+    <xacro:property name="lauv_cob" value="0 0 0.01"/>
     <!-- Vehicle's actual volume (Gazebo cannot compute the volume out of the mesh) -->
-    <xacro:property name="lauv_volume" value="0"/>
+    <xacro:property name="lauv_volume" value="0.017551374956865266"/>
     <!-- Describing the dimensions of the vehicle's bounding box -->
-    <xacro:property name="lauv_length" value="0"/>
-    <xacro:property name="lauv_width"  value="0"/>
-    <xacro:property name="lauv_height" value="0"/>
+    <xacro:property name="lauv_length" value="1.08"/>
+    <xacro:property name="lauv_width"  value="0.15"/>
+    <xacro:property name="lauv_radius"  value="${0.5 * lauv_width}"/>
+    <xacro:property name="lauv_height" value="0.15"/>
     <xacro:macro name="lauv_hydro_model" params="namespace">
       <!-- List of hydrodynamic models this robot's links -->
@@ -26,21 +27,14 @@
         <!-- Center of buoyancy -->
         <center_of_buoyancy>${lauv_cob}</center_of_buoyancy>
-        <!--
-        Choose one of the hydrodynamic models below, all are based on
-        Fossen's equation of motion for underwater vehicles
-        Reference:
-        [1] Fossen, Thor I. Handbook of marine craft hydrodynamics and motion
-            control. John Wiley & Sons, 2011.
-        -->
         <!-- 1) Fossen's equation of motion -->
         <hydrodynamic_model>
           <type>fossen</type>
           <added_mass>
-            0 0 0 0 0 0
-            0 0 0 0 0 0
-            0 0 0 0 0 0
-            0 0 0 0 0 0
-            0 0 0 0 0 0
-            0 0 0 0 0 0
+            1     0     0     0     0     0
+            0     16    0     0     0     0
+            0     0     16    0     0     0
+            0     0     0     0.005 0     0
+            0     0     0     0     1.3   0
+            0     0     0     0     0     1.3
           </added_mass>
           <!--
@@ -49,5 +43,10 @@
           -->
           <linear_damping>
-            0 0 0 0 0 0
+            -2.4  0     0     0     0     0
+            0     -23   0     0     0     11.5
+            0     0     -23   0     -11.5 0
+            0     0     0     -0.3  0     0
+            0     0     3.1   0     -9.7  0
+            0     -3.1  0     0     0     -9.7
           </linear_damping>
           <!--
@@ -65,31 +64,11 @@
           -->
           <quadratic_damping>
-            0 0 0 0 0 0
+            -2.4   0      0      0       0      0
+            0      -80    0      0       0      0.3
+            0      0      -80    0       -0.3   0
+            0      0      0      -0.0006 0      0
+            0      0      1.5    0       -9.1   0
+            0      -1.5   0      0       0      -9.1
           </quadratic_damping>
-          <!--
-            In case you want to model a simple surface vessel, you can use the
-            implementation of linear (small angle) theory for boxed shaped vessels
-            by providing the following parameters. If you omit the area of the
-            water level plane area, it will be calculated from the bounding box
-            parameters. Uncomment the lines below in case you are simulating a
-            surface vessel.
-            For more details on these parameters and the computation of buoyancy
-            for vessels using this theory, check:
-              [1] Lecture Notes  TTK 4190 Guidance and Control of Vehicles (T. I. Fossen)
-                  http://www.fossen.biz/wiley/Ch4.pdf
-              [2] Fossen, Thor I. Handbook of marine craft hydrodynamics and motion
-                  control. John Wiley & Sons, 2011.
-          -->
-          <!--
-          <metacentric_width>0.0</metacentric_width>
-          <metacentric_length>0.0</metacentric_length>
-          <submerged_height>0.0</submerged_height>
-          -->
-        </hydrodynamic_model>
-        <!-- 2) This computes the added-mass and damping parameters for a sphere
-        in the fluid with the given radius -->
-        <hydrodynamic_model>
-          <type>sphere</type>
-          <radius>0</radius>
         </hydrodynamic_model>
       </link>

File: src/lauv_description/urdf/sensors.xacro (robot description, xacro)
@@ -10,28 +10,51 @@
   <xacro:default_gps namespace="${namespace}" parent_link="${namespace}/base_link" />
   <!-- Mount a Pose 3D sensor. -->
-  <xacro:default_pose_3d namespace="${namespace}" parent_link="${namespace}/base_link" />
+  <xacro:default_pose_3d_macro
+    namespace="${namespace}"
+    parent_link="${namespace}/base_link"
+    inertial_reference_frame="${inertial_reference_frame}" />
   <!-- Forward-looking sonar sensor -->
-  <xacro:forward_multibeam_p900 namespace="${namespace}" parent_link="${namespace}/base_link">
+  <!-- <xacro:forward_multibeam_p900 namespace="${namespace}" parent_link="${namespace}/base_link">
     <origin xyz="0 0 0" rpy="0 0 0"/>
-  </xacro:forward_multibeam_p900>
+  </xacro:forward_multibeam_p900> -->
   <!-- DVL  -->
-  <xacro:default_dvl namespace="${namespace}" parent_link="${namespace}/base_link">
+  <!-- <xacro:default_dvl namespace="${namespace}" parent_link="${namespace}/base_link">
     <origin xyz="0 0 0" rpy="0 0 0"/>
-  </xacro:default_dvl>
+  </xacro:default_dvl> -->
   <!-- RPT  -->
-  <xacro:default_rpt namespace="${namespace}" parent_link="${namespace}/base_link">
+  <!-- <xacro:default_rpt namespace="${namespace}" parent_link="${namespace}/base_link">
     <origin xyz="0 0 0" rpy="0 0 0"/>
-  </xacro:default_rpt>
+  </xacro:default_rpt> -->
   <!-- Pressure  -->
-  <xacro:default_pressure namespace="${namespace}" parent_link="${namespace}/base_link">
+  <!-- <xacro:default_pressure namespace="${namespace}" parent_link="${namespace}/base_link">
     <origin xyz="0 0 0" rpy="0 0 0"/>
-  </xacro:default_pressure>
+  </xacro:default_pressure> -->
   <!-- IMU  -->
   <xacro:default_imu namespace="${namespace}" parent_link="${namespace}/base_link">
     <origin xyz="0 0 0" rpy="0 0 0"/>
   </xacro:default_imu>
-  <!-- Mount a camera  -->
-  <xacro:default_camera namespace="${namespace}" parent_link="${namespace}/base_link" suffix="">
+  <!-- Mount a camera -->
+  <!-- <xacro:default_camera namespace="${namespace}" parent_link="${namespace}/base_link">
     <origin xyz="0 0 0" rpy="0 0 0"/>
-  </xacro:default_camera>
+  </xacro:default_camera> -->
+  <!-- Mount the chemical concentration sensor -->
+  <xacro:chemical_concentration_sensor_macro
+      namespace="${namespace}"
+      suffix=""
+      reference_frame="world"
+      parent_link="${namespace}/base_link"
+      input_topic="/plume/particles"
+      output_topic="particle_concentration"
+      update_rate="2"
+      gamma="0.001"
+      water_salinity_value="35.0"
+      plume_salinity_value="1.0"
+      salinity_output_topic="salinity"
+      salinity_unit="ppt"
+      gain="5.0"
+      noise_sigma="0.01"
+      noise_amplitude="1"
+      radius="50.0">
+    <origin xyz="0 0 0" rpy="0 0 0"/>
+  </xacro:chemical_concentration_sensor_macro>
 </robot>
